File: hardware/4x4 v2/4x4v3.sch (EAGLE design)
At the start: 59 parts, among them IC1 PIC18F2480-I/SP, J1 USB1035-XX-X-X-X-B_REVE, T1 BC547, T2 BC547, T3 BC547, T4 BC547, U1 IR3315, U2 IR3315, U3 IR3315, U4 IR3315

Commit message: Rev
Parts:
- removed 12V-1: GMSTBA2, con-phoenix-762:GMSTBA2
- removed J1: USB1035-XX-X-X-X-B_REVE, USB1035-XX-X-X-X-B_REVE:USB1035-XX-X-X-X-B_REVE
- removed LED4: (no value), led:LEDCHIP-LED0805
- removed LED6, LED7, LED8: (no value), led:LEDCHIPLED_0805
- removed R11: 680, resistor:R-US_R0805
- removed R19, R21, R23: (no value), resistor:R-US_R0805
- added 12V-IN-1: MSTBV4, con-phoenix-508:MSTBV4
- added J2: (no value), InputOutputIO (rev17e):614008235023
- added JP4, JP5: (no value), pinhead:PINHD-2X3
- added R24: 10k, resistor:R-US_R0805
- added R27: 100R, resistor:R-US_R0805
- C1: value (none) -> 0.1uF
- C2: value (none) -> 100nF; device resistor:C-EU050-035X075 -> resistor:C-EU025-025X050
- IN-1, OUT-1: value MSTBA4 -> MSTBV4; device con-phoenix-508:MSTBA4 -> con-phoenix-508:MSTBV4
- JP1: value (none) -> ICSP
- JP2: value (none) -> 5V REG
- JP3: value (none) -> 5V USB
- LED1: value 12123 -> (none); device led:LEDCHIP-LED0805 -> led:LEDCHIPLED_0805
- LED2, LED3: device led:LEDCHIP-LED0805 -> led:LEDCHIPLED_0805
- R14, R5, R8: value 680 -> (none)
- R25: value (none) -> 150R
- R3: value (none) -> 10k
- S1: value (none) -> KMR421GULCLFS; device switch-omron:10-XX -> KMR421GULCLFS:KMR421GULCLFS
Connections:
- removed net N$11: LED4.C, R14.1
- removed net N$14: LED5.C, R17.2
- removed net N$17: LED6.C, R19.2
- removed net N$20: LED7.C, R21.2
- removed net N$23: LED8.C, R23.2
- new net N$3: LED5.A, R1.2
- new net SCL: IC1.RC3/SCK/SCL, JP4.4, JP5.4, R17.1
- new net SDA: IC1.RC4/SDI/SDA, JP4.2, JP5.2, R14.2
- net 12V-1: now also 12V-IN-1-2.1, 12V-IN-1-3.1; no longer 12V-1-2.1
- net GND: now also 12V-IN-1-1.1, 12V-IN-1-4.1, J2.A_GND, J2.A_SHIELD, J2.B_GND, J2.B_SHIELD, JP4.3, JP5.3, LED1.C, LED2.C, LED3.C, LED5.C, R27.1, S1.G; no longer 12V-1-1.1, J1.GND1, J1.GND2, J1.SHIELD, R11.2, R14.2, R17.1, R19.1, R21.1, R23.1, R3.1, R5.2, R8.2
- net IN-1-1: now also R1.1; no longer LED1.A
- net IN-1-2: now also R2.1; no longer LED2.A
- net IN-1-3: now also R5.1; no longer LED3.A
- net IN-1-4: now also R8.1; no longer LED4.A
- net MCLR: now also R3.1; no longer R1.1
- net N$1: now also R24.1, R3.2, S1.3; no longer R1.2, R2.1, S1.S
- net N$2: now also R27.2, S1.1; no longer R3.2, S1.P
- net N$5: now also LED1.A, R2.2; no longer LED1.C, R5.1
- net N$7: now also LED2.A, R5.2; no longer LED2.C, R8.1
- net N$9: now also LED3.A, R8.2; no longer LED3.C, R11.1
- net OUT-1-5: now also J2.A_VBUS, J2.B_VBUS; no longer J1.VBUS1, J1.VBUS2
- net SIGIN-1-1: now also IC1.RC6/TX/CK; no longer IC1.RA0/AN0
- net SIGIN-1-2: now also IC1.RC7/RX/DT; no longer IC1.RA1/AN1
- net SIGIN-1-3: now also IC1.INT0/AN10/RB0; no longer IC1.RA2/AN2/VREF-
- net SIGIN-1-4: now also IC1.INT1/AN8/RB1; no longer IC1.RA3/AN3/VREF+
- net SIGOUT-1-1: now also IC1.KBI1/PGM/RB5; no longer IC1.INT1/AN8/RB1, LED5.A
- net SIGOUT-1-2: now also IC1.KBI0/AN9/RB4; no longer IC1.INT2/CANTX/RB2, LED6.A
- net SIGOUT-1-3: no longer LED7.A
- net SIGOUT-1-4: now also IC1.INT2/CANTX/RB2; no longer IC1.KBI0/AN9/RB4, LED8.A
- net SIGOUT-1-5: now also IC1.RA0/AN0; no longer IC1.KBI1/PGM/RB5
- net VCC: now also JP4.1, JP5.1, R14.1, R17.2, R24.2; no longer R2.2
