File: hardware/Expansion v3/Expansionv3.sch (EAGLE design)
At the start: 55 parts, among them IC1 PIC18F2480-I/SP, T1 BC547, T2 BC547, T3 BC547, T4 BC547, U1 IR3315, U2 IR3315, U3 IR3315, U4 IR3315

Commit message: Added ext board
Parts:
- removed C1: 0.1uF, resistor:C-EU025-030X050
- removed C2: 100nF, resistor:C-EU025-025X050
- removed JP1: ICSP, pinhead:PINHD-1X6
- removed JP2: 5V REG, pinhead:PINHD-1X3
- removed LED10: (no value), led:LEDCHIPLED_0805
- removed LED9: STATUS, led:LEDCHIPLED_0805
- removed R14, R26: (no value), resistor:R-US_R0805
- removed R24, R3: 10k, resistor:R-US_R0805
- removed R25: 150R, resistor:R-US_R0805
- removed R27: 100R, resistor:R-US_R0805
- added R19, R21: (no value), resistor:R-US_R0805
- IC1: value PIC18F2480-I/SP -> PCF8574P; device microchip:PIC18F2480-I/SP -> micro-philips:PCF8574P
- S1: value KMR421GULCLFS -> SWS003; device KMR421GULCLFS:KMR421GULCLFS -> smd-special:SWS003
- renumbered 12V-IN-1 to 12V-IN, IN-1 to IN, OUT-1 to OUT
Connections:
- net IN-1-1 renamed IN-1
- net IN-1-2 renamed IN-2
- net IN-1-3 renamed IN-3
- net IN-1-4 renamed IN-4
- net OUT-1-1 renamed OUT-1
- net OUT-1-2 renamed OUT-2
- net OUT-1-3 renamed OUT-3
- net OUT-1-4 renamed OUT-4
- net OUT-1-5 renamed OUT-5
- removed net 12V-1: 12V-IN-2.1, 12V-IN-3.1, JP2.1, JP3.3, LED10.A, U1.VCC, U2.VCC, U3.VCC, U4.VCC
- removed net MCLR: IC1.RE3/!MCLR/VPP, JP1.1, R3.1
- removed net N$1: C2.1, R24.1, R3.2, S1.3
- removed net N$2: R27.2, S1.1
- removed net N$24: LED9.A, R25.2
- removed net N$25: LED10.C, R26.1
- removed net PGC: IC1.KBI2/PGC/RB6, JP1.5
- removed net PGD: IC1.KBI3/PGD/RB7, JP1.4
- removed net PGM: JP1.6
- removed net SIGIN-1-1: IC1.RC6/TX/CK, R6.2, T1.C
- removed net SIGIN-1-2: IC1.RC7/RX/DT, R9.2, T2.C
- removed net SIGIN-1-3: IC1.INT0/AN10/RB0, R12.2, T3.C
- removed net SIGIN-1-4: IC1.INT1/AN8/RB1, R15.2, T4.C
- removed net SIGOUT-1-1: IC1.KBI1/PGM/RB5, T5.B
- removed net SIGOUT-1-2: IC1.KBI0/AN9/RB4, T6.B
- removed net SIGOUT-1-3: IC1.CANRX/RB3, T7.B
- removed net SIGOUT-1-4: IC1.INT2/CANTX/RB2, T8.B
- removed net SIGOUT-1-5: IC1.RA0/AN0, T9.B
- removed net STATUS_LED: IC1.RC1/T1OSI, R25.1
- new net 12V: 12V-IN-2.1, 12V-IN-3.1, JP3.3, U1.VCC, U2.VCC, U3.VCC, U4.VCC
- new net A0: IC1.A0, R21.2, S1.1
- new net A1: IC1.A1, R19.2, S1.2
- new net A2: IC1.A2, R17.2, S1.3
- new net INT: IC1.!INT, JP4.5, JP5.5
- new net SIGIN-1: IC1.P0, R6.2, T1.C
- new net SIGIN-2: IC1.P1, R9.2, T2.C
- new net SIGIN-3: IC1.P2, R12.2, T3.C
- new net SIGIN-4: IC1.P3, R15.2, T4.C
- new net SIGOUT-1: IC1.P4, T5.B
- new net SIGOUT-2: IC1.P5, T6.B
- new net SIGOUT-3: IC1.P6, T7.B
- new net SIGOUT-4: IC1.P7, T8.B
- new net SIGOUT-5: T9.B
- net GND: now also R17.1, R19.1, R21.1; no longer C1.2, C2.2, IC1.VSS@1, JP1.3, JP2.2, LED9.C, R26.2, R27.1, S1.G
- net SCL: now also IC1.SCL; no longer IC1.RC3/SCK/SCL, R17.1
- net SDA: now also IC1.SDA; no longer IC1.RC4/SDI/SDA, R14.2
- net VCC: now also S1.4, S1.5, S1.6; no longer C1.1, JP1.2, JP2.3, R14.1, R17.2, R24.2
Other:
- moved on the sheet: R17
